Commit message: HSL26: лабиринт lab1/lab2/template, second-robot спавн, launch-параметризация
- worlds/{lab1,lab2,template,empty}.world — Gazebo-миры лабиринта
  (Labirint_bez_prepyatstviy.zip как источник), lab1 теперь дефолт,
  с двумя выходами (Wall_144/Wall_117 удалены)
- gazebo.launch.py: аргументы world/lidar_samples/spawn_x/spawn_y/spawn_yaw,
  плюс спавн второго робота (та же модель, все <gazebo>-плагины вырезаны
  из URDF перед спавном — иначе делил бы с роботом А глобальные топики
  диффдрайва/IMU/лидара, т.к. namespace ещё не реализован)
- mast.urdf.xacro: xacro:arg lidar_samples (регулируемая плотность скана)
- README.md, Reglament_HSL26_-_v06092026.pdf — регламент нового этапа
- CLAUDE.md — конспект всей сессии: находки по Gazebo/лидару, переход
  HSL25 -> HSL26

File: hsl_description/urdf/mast.urdf.xacro (robot description, xacro)
@@ -230,14 +230,18 @@
     <xacro:property name="lidar_publish_rate" value="10"/>
     <!-- Из реального bag-файла (data/rosbag2_..._static_1m) настоящий
-         livox/lidar даёт ~20000 точек/сообщение на ~8.5Гц. Подобрано
-         эмпирически (ros2 topic hz + сравнение /clock с wall-time):
-         10000 — разумный баланс (реальная частота ~30Гц, real-time factor
-         ~0.68); на 20000 совокупная пропускная способность НЕ растёт (сама
-         частота падает непропорционально сильнее — ~2.7Гц, деградация
-         нелинейная), только просаживает производительность и время
-         старта. Меньше половины точек реального робота на скан, но не
-         из экономии, а потому что 20000 объективно не имеет смысла при
-         текущей производительности плагина. -->
-    <xacro:property name="lidar_samples" value="10000"/>
+         livox/lidar даёт ~20000 точек/сообщение на ~8.5Гц. На 10000 —
+         real-time factor ~0.68; на 20000 совокупная пропускная способность
+         НЕ растёт (частота падает непропорционально сильнее — ~2.7Гц),
+         только просаживает производительность и время старта. Но 10000
+         (и тем более 20000) — это уже при полностью свободном CPU;
+         под обычной десктопной нагрузкой (браузер/IDE и т.п.) плагин
+         (однопоточный, без защиты от отставания) начинает копить лаг между
+         облаком и текущей позицией робота в несколько секунд — см. CLAUDE.md,
+         "Message Filter... timestamp is earlier than all data in cache".
+         Задаётся launch-аргументом `lidar_samples` в gazebo.launch.py
+         (дефолт снижен до 2000 именно из-за этого — быстрее реагирует,
+         компромисс по плотности облака) — менять там, а не здесь. -->
+    <xacro:arg name="lidar_samples" default="2000"/>
+    <xacro:property name="lidar_samples" value="$(arg lidar_samples)"/>
     <xacro:property name="lidar_downsample" value="1"/>
     <xacro:property name="lidar_noise_stddev" value="0.0"/>
