Commit message: Реалистичная одометрия и шум сенсоров + запуск SLAM одной командой
ОДОМЕТРИЯ. /odom был ground truth прямо из физики Gazebo: у плагина
diff_drive дефолт odometry_source=WORLD, а тег не был задан. Живой тест:
робот упёрт в стену, колёса накрутили 1.17 м, /odom сдвинулся на 0.0008 м -
для энкодеров невозможно. SLAM получал недрейфующий prior и scan matching
фактически не проверялся (коррекция map->odom 3 см за прогон).

Теперь как у реального kobuki_node (kobuki_node/src/odometry.cpp):
- odometry_source=0 (счисление по колёсам), publish_odom_tf=false,
  сырая одометрия уходит на _raw/odom
- новый scripts/odometry_bridge.py: x,y от энкодеров, yaw и angular.z
  перезаписываются гироскопом (use_imu_heading: true в конфиге
  организаторов), публикует odom + TF odom->base_link, covariance как у
  драйвера
Проверка: в упоре энкодеры "повернули" робота на -50.6 град, гироскоп
показал +0.2 град - /odom отдаёт правду. Коррекция map->odom выросла до
2.26 м, ошибка локализации SLAM против физики 6 см.

ШУМ СЕНСОРОВ. Два бага по дороге:
- старый формат <imu><noise><rate>/<accel> современный Gazebo МОЛЧА
  игнорирует (с bias_mean=0.1 рад/с показания оставались ~0.00005);
  переведено на поосевой <angular_velocity><x><noise>
- Gazebo не применяет шум к orientation, поэтому gyro_imu_bridge.py
  теперь ИНТЕГРИРУЕТ угловую скорость в курс - как прошивка kobuki
  (inertia.data.angle). Замер ухода курса: +0.32 град/мин

Значения измерены по реальной записи квалификации (static_1m), а не взяты
из даташита: лидар 0.005 м (фит плоскости стены на 1/2/3 м), Livox IMU
0.0015 рад/с и 0.076 м/с². Гироскоп kobuki - оценка, его нет в записях.
lidar_noise_stddev вынесен в аргумент launch (0.0 возвращает ground truth).

SLAM. Добавлен robot_slam/launch/gazebo_slam_mapping.launch.py - двойник
плюс построение карты одной командой, через IncludeLaunchDescription на
уже существующие gazebo.launch.py и slam.launch.py. Из gazebo.launch.py
убраны 3 ноды локализации, вставленные туда вручную: они дублировали
robot_slam/launch/localization.launch.py, и при запуске второго launch
получались две ноды с одинаковыми именами (livox_to_livox_frame,
pointcloud_to_laserscan, slam_toolbox) плюс два slam_toolbox, спорящих за
публикацию TF map->odom. Теперь удалять ноды руками не нужно:
gazebo.launch.py + localization.launch.py ИЛИ slam.launch.py.

Co-Authored-By: Claude Opus 5 <noreply@anthropic.com>

File: hsl_description/urdf/kobuki_gazebo.urdf.xacro (robot description, xacro)
@@ -166,21 +166,23 @@
         <frame_name>gyro_link</frame_name>
         <visualize>false</visualize>
+        <!-- ⚠️⚠️ ФОРМАТ ВАЖЕН: старый <imu><noise><rate>/<accel> (он тут и
+             стоял, унаследован из апстрима kobuki_description) современный
+             Gazebo МОЛЧА ИГНОРИРУЕТ — проверено вживую: с bias_mean=0.1
+             рад/с показания оставались ~0.00005, шума не было вообще.
+             Рабочий формат — поосевой <angular_velocity><x><noise>.
+             Значения: stddev 0.0044 рад/с = 0.25 град/с (то, что и имел в
+             виду комментарий в старом блоке, но записанное там
+             ${0.0014*0.0014} давало ~2e-6 — похоже на случайный квадрат).
+             bias_stddev 0.0005 рад/с — это ОЦЕНКА, а не замер: гироскопа
+             базы kobuki нет в bag-записях квалификации (там только
+             /livox/lidar и /livox/imu). Порядок подобран так, чтобы курс
+             уходил примерно на 1-2 град/мин, как у реального kobuki. -->
         <imu>
-          <noise>
-            <type>gaussian</type>
-	          <rate>
-	            <mean>0.0</mean>
-	            <stddev>${0.0014*0.0014}</stddev> <!-- 0.25 x 0.25 (deg/s) -->
-	            <bias_mean>0.0</bias_mean>
-	            <bias_stddev>0.0</bias_stddev>
-	          </rate>
-		        <accel> <!-- not used in the plugin and real robot, hence using tutorial values -->
-			        <mean>0.0</mean>
-			        <stddev>1.7e-2</stddev>
-			        <bias_mean>0.1</bias_mean>
-			        <bias_stddev>0.001</bias_stddev>
-		        </accel>
-          </noise>
-	      </imu>
+          <angular_velocity>
+            <x><noise type="gaussian"><mean>0.0</mean><stddev>0.0044</stddev><bias_mean>0.0</bias_mean><bias_stddev>0.0005</bias_stddev></noise></x>
+            <y><noise type="gaussian"><mean>0.0</mean><stddev>0.0044</stddev><bias_mean>0.0</bias_mean><bias_stddev>0.0005</bias_stddev></noise></y>
+            <z><noise type="gaussian"><mean>0.0</mean><stddev>0.0044</stddev><bias_mean>0.0</bias_mean><bias_stddev>0.0005</bias_stddev></noise></z>
+          </angular_velocity>
+        </imu>
       </sensor>
 	  </gazebo>
@@ -200,4 +202,9 @@
                (см. kobuki_node/src/kobuki_ros.cpp:168) -->
           <remapping>cmd_vel:=commands/velocity</remapping>
+          <!-- Сырое счисление по энкодерам уходит на СКРЫТЫЙ топик, не для
+               прямого использования командой. Итоговый "odom" (уже с курсом
+               от гироскопа, как у реального драйвера) публикует
+               scripts/odometry_bridge.py -->
+          <remapping>odom:=_raw/odom</remapping>
         </ros>
         <update_rate>10</update_rate>
@@ -210,10 +217,20 @@
         <!-- output -->
         <publish_odom>true</publish_odom>
-        <publish_odom_tf>true</publish_odom_tf>
+        <!-- ⚠️ TF odom->base_link НЕ от плагина: его публикует
+             odometry_bridge.py, иначе TF (с "сырым" энкодерным курсом) и
+             топик /odom (с курсом от гироскопа) разошлись бы между собой -->
+        <publish_odom_tf>false</publish_odom_tf>
         <publish_wheel_tf>true</publish_wheel_tf>
-        <!-- odom_publisher_ реального драйвера: nav_msgs/Odometry на "odom",
-             odom_frame="odom", base_frame="base_link" — уже совпадает
-             (см. kobuki_node_params.yaml); default-топик "odom" у плагина
-             и так верный, remapping не нужен -->
+        <!-- ⚠️⚠️ ODOMETRY_SOURCE=0 (ENCODER) — критично, дефолт плагина это
+             WORLD, т.е. поза берётся прямо из физики Gazebo и НЕ дрейфует
+             вообще. Проверено живым тестом: робот, упёртый в стену с
+             буксующими колёсами (накрутили 1.17м), давал смещение /odom
+             0.0008м — невозможное поведение для энкодеров, из-за чего SLAM
+             получал идеальный prior и scan matching фактически не
+             проверялся (коррекция map->odom 3см за прогон против 2.26м
+             после переключения). Реальный kobuki считает x,y именно
+             счислением по колёсам (kobuki_node/src/odometry.cpp,
+             ecl::extend_pose) -->
+        <odometry_source>0</odometry_source>
         <odometry_frame>odom</odometry_frame>
         <robot_base_frame>base_link</robot_base_frame>

File: hsl_description/urdf/mast.urdf.xacro (robot description, xacro)
@@ -189,20 +189,28 @@
         <update_rate>200</update_rate>
         <visualize>false</visualize>
+        <!-- ⚠️ Формат поосевой (<angular_velocity><x><noise>): старый
+             <imu><noise><rate>/<accel>, который тут стоял, современный
+             Gazebo молча игнорирует — см. подробности у гироскопа kobuki
+             в kobuki_gazebo.urdf.xacro.
+             Значения ИЗМЕРЕНЫ по реальной bag-записи квалификации
+             (data/rosbag2_2026_06_27-18_27-static_1m, робот неподвижен,
+             1992 сообщения /livox/imu):
+               gyro:  stddev 0.0011..0.0021 рад/с, смещения по осям
+                      +0.0151 / -0.0045 / -0.0005 рад/с
+               accel: stddev 0.0023..0.0077 g
+             accel здесь задаётся в м/с² (livox_imu_bridge.py делит на 9.81,
+             воспроизводя баг реального драйвера с единицами "g"):
+             0.0077 g * 9.81 = 0.076 м/с². -->
         <imu>
-          <noise>
-            <type>gaussian</type>
-            <rate>
-              <mean>0.0</mean>
-              <stddev>${0.0014*0.0014}</stddev>
-              <bias_mean>0.0</bias_mean>
-              <bias_stddev>0.0</bias_stddev>
-            </rate>
-            <accel>
-              <mean>0.0</mean>
-              <stddev>1.7e-2</stddev>
-              <bias_mean>0.1</bias_mean>
-              <bias_stddev>0.001</bias_stddev>
-            </accel>
-          </noise>
+          <angular_velocity>
+            <x><noise type="gaussian"><mean>0.0</mean><stddev>0.0015</stddev><bias_mean>0.0</bias_mean><bias_stddev>0.008</bias_stddev></noise></x>
+            <y><noise type="gaussian"><mean>0.0</mean><stddev>0.0015</stddev><bias_mean>0.0</bias_mean><bias_stddev>0.008</bias_stddev></noise></y>
+            <z><noise type="gaussian"><mean>0.0</mean><stddev>0.0015</stddev><bias_mean>0.0</bias_mean><bias_stddev>0.008</bias_stddev></noise></z>
+          </angular_velocity>
+          <linear_acceleration>
+            <x><noise type="gaussian"><mean>0.0</mean><stddev>0.076</stddev><bias_mean>0.0</bias_mean><bias_stddev>0.01</bias_stddev></noise></x>
+            <y><noise type="gaussian"><mean>0.0</mean><stddev>0.076</stddev><bias_mean>0.0</bias_mean><bias_stddev>0.01</bias_stddev></noise></y>
+            <z><noise type="gaussian"><mean>0.0</mean><stddev>0.076</stddev><bias_mean>0.0</bias_mean><bias_stddev>0.01</bias_stddev></noise></z>
+          </linear_acceleration>
         </imu>
       </sensor>
@@ -245,5 +253,14 @@
     <xacro:property name="lidar_samples" value="$(arg lidar_samples)"/>
     <xacro:property name="lidar_downsample" value="1"/>
-    <xacro:property name="lidar_noise_stddev" value="0.0"/>
+    <!-- Шум дальности лидара. ИЗМЕРЕН по реальной записи квалификации
+         (static_1m): фит плоскости стены дал stddev остатков 0.0049 / 0.0067
+         / 0.0043 м на дистанциях ~1 / ~2 / ~3 м -> ~0.005 м. Ноль здесь
+         означал бы идеально чистое облако, какого у реального MID-360 не
+         бывает; для robot_b_detector это важнее, чем для SLAM — его пороги
+         (inlier_thresh=0.02 у плоскости пола, voxel 0.03) подбирались на
+         реальных, шумных данных. lidar_noise_stddev:=0.0 возвращает
+         ground truth, если нужно сравнить. -->
+    <xacro:arg name="lidar_noise_stddev" default="0.005"/>
+    <xacro:property name="lidar_noise_stddev" value="$(arg lidar_noise_stddev)"/>
     <gazebo reference="lidar_mount_link">
       <sensor type="ray" name="livox">
